Commit message: Added settings for rick and morty styles

File: xacro/barista_robot_model.urdf.xacro (robot description, xacro)
@@ -3,4 +3,12 @@
     <!-- Arguments & Properties -->
     <xacro:arg name="include_laser" default="true" />
+    <xacro:arg name="robot_name" default="rick" />
+    <xacro:property name="robot_name" value="$(arg robot_name)" />
+    <xacro:property name="body_color" value="red" />
+    <xacro:property name="body_gz_material" value="Gazebo/Red"/>
+    <xacro:if value="${robot_name == 'morty'}">
+        <xacro:property name="body_color" value="blue" />
+        <xacro:property name="body_gz_material" value="Gazebo/Blue"/>
+    </xacro:if>
     <!-- Includes -->
     <xacro:include filename="$(find barista_robot_description)/xacro/materials.xacro" />
@@ -19,5 +27,5 @@
                 <cylinder length="0.155" radius="0.178"/>
             </geometry>
-            <material name="red"/>
+            <material name="${body_color}"/>
         </visual>
         <collision>
@@ -32,5 +40,5 @@
     </link>
     <gazebo reference="base_link">
-        <material>Gazebo/Red</material>
+        <material>${body_gz_material}</material>
     </gazebo>
     <joint name="base_footprint_joint" type="fixed">
@@ -74,8 +82,12 @@
         />
     <!-- Cup Holder Tray --> <!-- 0.0775 + 0.22 + 0.045-->
-    <xacro:cup_holder_tray name="cup_holder_tray" parent="base_link" xyz="0.0 0.0 0.3425" />
+    <xacro:cup_holder_tray name="cup_holder_tray"
+        parent="base_link"
+        xyz="0.0 0.0 0.3425"
+        color="${body_color}"
+        gz_material="${body_gz_material}" />
     <!-- Planar Laser Scanner -->
     <xacro:if value="$(arg include_laser)">
-        <xacro:laser_scanner name="laser_scan" parent="base_link" xyz="0.11 0.0 0.0775" />
+        <xacro:laser_scanner name="laser_scan" parent="base_link" xyz="0.11 0.0 0.0775" robot_name="${robot_name}" />
     </xacro:if>
     <!-- PLUGINS -->
@@ -84,4 +96,5 @@
         <plugin name="barista_robot_joint_state" filename="libgazebo_ros_joint_state_publisher.so">
             <ros>
+                <namespace>/${robot_name}</namespace>
                 <remapping>~/out:=joint_states</remapping>
             </ros>
@@ -100,4 +113,8 @@
     <gazebo>
         <plugin filename="libgazebo_ros_diff_drive.so" name="differential_drive_controller">
+            <ros>
+                <namespace>/${robot_name}</namespace>
+                <remapping>/cmd_vel:=cmd_vel</remapping>
+            </ros>
             <!-- wheels -->
             <left_joint>left_wheel_joint</left_joint>
@@ -112,6 +129,6 @@
             <publish_odom>true</publish_odom>
             <publish_odom_tf>true</publish_odom_tf>
-            <odometry_frame>odom</odometry_frame>
-            <robot_base_frame>base_footprint</robot_base_frame>
+            <odometry_frame>${robot_name}/odom</odometry_frame>
+            <robot_base_frame>${robot_name}/base_footprint</robot_base_frame>
         </plugin>
     </gazebo>

File: xacro/cup_holder_tray.xacro (robot description, xacro)
@@ -5,5 +5,5 @@
     <xacro:property name="cup_holder_length" value="0.09" />
     <!-- Cup Holder Tray Wheel Macro -->
-    <xacro:macro name="cup_holder_tray" params="name parent xyz">
+    <xacro:macro name="cup_holder_tray" params="name parent xyz color gz_material">
        <link name="${name}">
             <visual>
@@ -11,5 +11,5 @@
                     <cylinder length="${cup_holder_length}" radius="${cup_holder_radius}"/>
                 </geometry>
-                <material name="red"/>
+                <material name="${color}"/>
             </visual>
             <collision>
@@ -28,5 +28,5 @@
         </link>
         <gazebo reference="${name}">
-            <material>Gazebo/Red</material>
+            <material>${gz_material}</material>
         </gazebo>
         <joint name="${name}_joint" type="fixed">

File: xacro/laser_scanner.xacro (robot description, xacro)
@@ -5,5 +5,5 @@
     <xacro:property name="laser_scan_height" value="0.07"/>
     <xacro:property name="laser_scan_mass" value="0.13" />
-    <xacro:macro name="laser_scanner" params="name parent xyz">
+    <xacro:macro name="laser_scanner" params="name parent xyz robot_name">
         <link name="${name}">
             <visual>
@@ -73,8 +73,9 @@
                 <plugin name="laser" filename="libgazebo_ros_ray_sensor.so">
                     <ros>
+                        <namespace>${robot_name}</namespace>
                         <remapping>~/out:=scan</remapping>
                     </ros>
                     <output_type>sensor_msgs/LaserScan</output_type>
-                    <frame_name>${name}_frame</frame_name>
+                    <frame_name>${robot_name}/${name}_frame</frame_name>
                 </plugin>
             </sensor>
